File: hall-sensor.kicad_pcb (KiCad board)
At the start: 2 copper layers, 15 x 15 mm, 7 parts, among them J1 SJ2-35464B-SMT-TR, U2 A31010SEHALT-10

Commit message: Update Library
Parts:
- C1: footprint Capacitor_SMD:C_0603_1608Metric -> V2_Capacitor_SMD:C_0603
- FID1: value Fiducial -> Fiducial_Paste
- H1, H2: value MountingHole_2.5mm -> 2.5mm
Routing:
- net GND: track 4.13 -> 4.81 mm
