File: hall-sensor.kicad_sch (KiCad schematic)
At the start: 7 parts, among them J1 SJ2-35464B-SMT-TR, U2 A31010SEHALT-10

Commit message: Update Library
Parts:
- C1: footprint Capacitor_SMD:C_0603_1608Metric -> V2_Capacitor_SMD:C_0603; symbol Device:C_Small -> V2_Capacitor:0603_0u1; Manufacturer (none) -> TDK; Mouser (none) -> 810-CGA3E2X7R1H104MA; Product (none) -> CGA3E2X7R1H104M080AA; Rating (none) -> 50V
- FID1: value Fiducial -> Fiducial_Paste
- H1, H2: value MountingHole_2.5mm -> 2.5mm
- J1: Manufacturer (none) -> Same Sky; Mouser (none) -> 490-SJ2-35464BSMT-TR; Product (none) -> SJ2-35464B-SMT-TR
- U2: Manufacturer (none) -> Allegro MicroSystems; Mouser (none) -> 250-A31010SEHALT-10; Product (none) -> A31010SEHALT-10
Other:
- moved on the sheet: FID1, H1, H2

Commit message: Good Bye Imperial
Parts:
- C1: footprint V2_Capacitor_SMD:C_0603 -> V2_Capacitor_SMD:C_1608; symbol V2_Capacitor:0603_0u1 -> V2_Capacitor:1608_0u1
Changed lines of the file:
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@@
 	)
 	(symbol
-		(lib_id "V2_Capacitor:0603_0u1")
+		(lib_id "V2_Capacitor:1608_0u1")
 		(at 205.74 105.41 0)
 		(unit 1)
@@
 			)
 		)
-		(property "Footprint" "V2_Capacitor_SMD:C_0603"
+		(property "Footprint" "V2_Capacitor_SMD:C_1608"
 			(at 205.74 122.428 0)
 			(effects
